Commit message: Exporter: Jazzy + Gz Harmonic-ready output
URDF body:
  - rename UrdfSerializer -> XacroGenerator
  - new SerializeBodyForRobot(model, root): prepend world link + fixed joint
    so the robot is anchored on spawn (was falling in Gz)
  - default zero effort/velocity joint limits to 100 / 1.0 (ros2_control +
    Gz reject zero); SerializeBody(model) untouched for golden tests

Launch:
  - single chained gz_sim.launch.py: gz + rsp + spawn + bridge + JSB->JTC
    spawners via OnProcessExit. Gz viewport is the only 3D view
  - drop display.launch.py, ros2_control.launch.py, rviz.rviz from the
    Robot Package writer

Wizard (Joints step):
  - MateInfo carries the two top-level component link names so the mate
    list filters to the active joint's pair
  - listbox-event guard prevents repopulate from auto-assigning the first
    visible mate to the joint (was breaking Next)
  - mate-highlight reverted to per-entity Select4 with diagnostic logging
    (Component2.Select4 was selecting whole components and corrupting
    Step 2 Links picker)

examples/: swap stale three_dof_arm_ros2 for fresh full_arm_ws export

File: examples/full_arm_ws/src/full_arm/urdf/inc/materials.xacro (robot description, xacro)
@@ -1,4 +1,4 @@
 <?xml version="1.0"?>
 <robot xmlns:xacro="http://www.ros.org/wiki/xacro">
-  <!-- Named materials populated by SW2GZ. -->
+  <!-- No named materials defined. -->
 </robot>

File: examples/full_arm_ws/src/full_arm/urdf/inc/ros2_control.xacro (robot description, xacro)
@@ -4,6 +4,7 @@
     <hardware>
       <plugin>gz_ros2_control/GazeboSimSystem</plugin>
+      <parameters>$(find full_arm)/config/controllers.yaml</parameters>
     </hardware>
-    <joint name="shoulder">
+    <joint name="link1_1_link1_2_joint">
       <command_interface name="position"/>
       <state_interface name="position"/>
@@ -11,11 +12,5 @@
       <state_interface name="effort"/>
     </joint>
-    <joint name="elbow">
-      <command_interface name="position"/>
-      <state_interface name="position"/>
-      <state_interface name="velocity"/>
-      <state_interface name="effort"/>
-    </joint>
-    <joint name="wrist">
+    <joint name="link1_2_link1_3_joint">
       <command_interface name="position"/>
       <state_interface name="position"/>
@@ -24,8 +19,3 @@
     </joint>
   </ros2_control>
-  <gazebo>
-    <plugin filename="gz_ros2_control-system" name="gz_ros2_control::system">
-      <parameters>$(find-pkg-share $(arg pkg))/config/controllers.yaml</parameters>
-    </plugin>
-  </gazebo>
 </robot>
